File: partner_video/dma.kicad_sch (KiCad schematic)
At the start: 3 parts, among them U30 8257, U40 MC8T97P (74LS367), U45 74LS244

Commit message: Update custom symbol attributes
Parts:
- U30: footprint Package_DIP:DIP-40_W15.24mm -> (none)
Changed lines of the file:
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@@
       (effects (font (size 1.27 1.27)) (justify left))
     )
-    (property "Footprint" "Package_DIP:DIP-40_W15.24mm" (at 110.49 92.71 0)
+    (property "Footprint" "" (at 110.49 92.71 0)
       (effects (font (size 1.27 1.27)) hide)
     )
-    (property "Datasheet" "https://pdos.csail.mit.edu/6.828/2012/readings/hardware/8237A.pdf" (at 110.49 90.17 0)
+    (property "Datasheet" "http://www.eecs.northwestern.edu/~ypa448/Microp/8257.pdf" (at 110.49 90.17 0)
       (effects (font (size 1.27 1.27)) hide)
     )
